File: Electronics/lcd13264-module/lcd13264-module.brd (EAGLE design)
At the start: 75.2 x 45.7 mm, 40 parts, among them J1 MICRO-SDCARD-CONNECTOR-330006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, U4 MIC5219-3.3V, X1 FH12-12S-1S, Y1 RESONATORSMD

Commit message: Unknown changes.
Parts:
- removed D1, D3: (no value), SparkFun-LED:LED-0603
- removed R1, R2: 1.5k, PaxInstrument-T400:SPARKFUN-RESISTORS_0603-RES
- moved ICSP2 33.1 mm to (14.0, 8.89), turned to 270 degrees
- moved ICSP1 27.4 mm to (14.0, 16.5), turned to 270 degrees
- moved C36 11.5 mm to (44.5, 22.9)
- moved R19 10.2 mm to (34.3, 24.1)
- moved C35 5.24 mm to (41.9, 22.9)
Connections:
- net DATA1 renamed D4/A6
- net DATA10 renamed D11
- net DATA2 renamed D9/A8
- net DATA3 renamed D12/A10
- net DATA4 renamed D8
- net DATA5 renamed D6/A7
- net DATA6 renamed D10
- net DATA7 renamed D5
- net DATA9 renamed D7
- net SCL renamed D3/SCL
- net SDA renamed D2/SDA
- removed net DATA8: U$3.32
- removed net LCD_MOSI: U$3.36, X1.6
- removed net LCD_SCK: U$3.37, X1.7
- removed net N$10: D1.A, R2.1
- removed net N$2: D3.C, U$3.21
- removed net N$37: C35.1, X1.3
- removed net N$39: C36.2, X1.1
- removed net N$5: D1.C, U$3.20
- removed net N$7: D3.A, R1.1
- new net A0: U$3.36
- new net A1: U$3.37
- new net A2: U$3.38
- new net D0: U$3.20
- new net D1: U$3.21
- new net N$11: C35.1, X1.10
- new net N$12: C36.2, X1.12
- net 3.3V: now also X1.1, X1.8; no longer R1.2, R2.2, X1.12, X1.5
- net GND: now also X1.9; no longer X1.4
- net LCD_A0: now also U$3.41, X1.5; no longer U$3.38, X1.8
- net LCD_BL: now also U$3.32; no longer U$3.41
- net LCD_CS: now also X1.3; no longer X1.10
- net LCD_RST: now also X1.4; no longer X1.9
- net MOSI: now also X1.7
- net N$38: now also X1.11; no longer X1.2
- net N$4: now also X1.2; no longer X1.11
- net SCK: now also X1.6
Routing:
- net D11: track 54.4 -> 22.0 mm
- net D5: track 36.7 -> 7.44 mm
- net 3.3V: track 164.3 -> 137.3 mm, vias 13 -> 12
- net D7: track 46.3 -> 20.2 mm
- net D3/SCL: track 57.0 -> 31.8 mm
- net D10: track 30.3 -> 8.60 mm
- net D2/SDA: track 44.7 -> 27.5 mm
- net D6/A7: track 26.8 -> 10.7 mm
- net D12/A10: track 24.3 -> 10.7 mm
- net LCD_MOSI: track 13.3 -> 0.00 mm
- net LCD_SCK: track 12.6 -> 0.00 mm
- net D8: track 22.1 -> 10.6 mm
- net D4/A6: track 21.7 -> 11.1 mm
- net LCD_A0: track 11.8 -> 2.27 mm
- net N$2: track 8.96 -> 0.00 mm
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