File: Electronics/lcd13264-module/lcd13264-module.sch (EAGLE design)
At the start: 39 parts, among them J1 MICRO-SDCARD-CONNECTOR-330006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, U4 MIC5219-3.3V, X1 FH12-12S-1S, Y1 RESONATORSMD

Commit message: Unknown changes.
Parts:
- removed D1, D3: (no value), SparkFun-LED:LED0603
- removed R1, R2: 1.5k, PaxInstrument-T400:SPARKFUN-RESISTORS_RESISTOR0603-RES
Connections:
- net DATA1 renamed D4/A6
- net DATA10 renamed D11
- net DATA2 renamed D9/A8
- net DATA3 renamed D12/A10
- net DATA4 renamed D8
- net DATA5 renamed D6/A7
- net DATA6 renamed D10
- net DATA7 renamed D5
- net DATA9 renamed D7
- net SCL renamed D3/SCL
- net SDA renamed D2/SDA
- removed net DATA8: U$3.PC7
- removed net LCD_MOSI: U$3.PF7(ADC7), X1-6.1
- removed net LCD_SCK: U$3.PF6(ADC6), X1-7.1
- removed net N$10: D1.A, R2.1
- removed net N$2: D3.C, U$3.PD3(TX)
- removed net N$37: C35.1, X1-3.1
- removed net N$39: C36.2, X1-1.1
- removed net N$5: D1.C, U$3.PD2(RX)
- removed net N$7: D3.A, R1.1
- new net A0: U$3.PF7(ADC7)
- new net A1: U$3.PF6(ADC6)
- new net A2: U$3.PF5(ADC5)
- new net D0: U$3.PD2(RX)
- new net D1: U$3.PD3(TX)
- new net N$11: C35.1, X1-10.1
- new net N$12: C36.2, X1-12.1
- net 3.3V: now also X1-1.1, X1-8.1; no longer R1.2, R2.2, X1-12.1, X1-5.1
- net GND: now also X1-9.1; no longer X1-4.1
- net LCD_A0: now also U$3.PF0(ADC0), X1-5.1; no longer U$3.PF5(ADC5), X1-8.1
- net LCD_BL: now also U$3.PC7; no longer U$3.PF0(ADC0)
- net LCD_CS: now also X1-3.1; no longer X1-10.1
- net LCD_RST: now also X1-4.1; no longer X1-9.1
- net MOSI: now also X1-7.1
- net N$38: now also X1-11.1; no longer X1-2.1
- net N$4: now also X1-2.1; no longer X1-11.1
- net SCK: now also X1-6.1
Other:
- moved on the sheet: X1-1, X1-10, X1-11, X1-12, X1-2, X1-3, X1-4, X1-5, X1-6, X1-7, X1-8, X1-9
